Commit message: Add robot meshes, add simulation support, update instructions

File: src/inmoov_description/robots/inmoov_head_control.urdf.xacro (robot description, xacro)
@@ -74,5 +74,4 @@
   </joint>
   <xacro:head covers="yes" />
-  <xacro:head_jaw covers="yes" />
   <xacro:face covers="yes" />
   <joint name="face_joint" type="fixed">

File: src/inmoov_description/urdf/asmHead.urdf.xacro (robot description, xacro)
@@ -1,4 +1,14 @@
 <?xml version="1.0"?>
 <robot name="inmoov" xmlns:xacro="http://ros.org/wiki/xacro">
+<link name="head_link">
+  <visual>
+    <geometry>
+      <mesh filename="package://inmoov_meshes/meshes/head.stl" scale="0.001 0.001 0.001"/>
+    </geometry>
+    <origin rpy="0 0 0" xyz="0 0 0"/>
+    <xacro:frame_color/>
+  </visual>
+  <xacro:head_inertial/>
+</link>
 <xacro:macro name="head" params="covers">
   <link name="head_base_link">
@@ -11,24 +21,4 @@
     </visual>
     <xacro:head_base_inertial/>
-  </link>
-  <link name="head_link">
-    <visual>
-      <geometry>
-        <mesh filename="package://inmoov_meshes/meshes/head.stl" scale="0.001 0.001 0.001"/>
-      </geometry>
-      <origin rpy="0 0 0" xyz="0 0 0"/>
-      <xacro:frame_color/>
-    </visual>
-    <xacro:head_inertial/>
-  </link>
-  <link name="jaw_link">
-    <visual>
-      <geometry>
-        <mesh filename="package://inmoov_meshes/meshes/jaw.stl" scale="0.001 0.001 0.001"/>
-      </geometry>
-      <origin rpy="0 0 0" xyz="0 0 0"/>
-      <xacro:cover_color/>
-    </visual>
-    <xacro:jaw_inertial/>
   </link>
   <link name="skull_link">
@@ -62,4 +52,5 @@
     <xacro:earrightv1_inertial/>
   </link>
+  <!-- See http://wiki.ros.org/urdf/XML/joint -->
   <joint name="head_pan_joint" type="revolute">
    <axis xyz="0 0 1"/>
@@ -68,11 +59,4 @@
    <parent link="head_base_link"/>
    <child link="head_link"/>
-  </joint>
-  <joint name="jaw_joint" type="revolute">
-   <axis xyz="0 1 0"/>
-   <limit effort="1000.0" lower="${jaw_joint_lower}" upper="${jaw_joint_upper}" velocity="${jaw_joint_velocity}" />
-   <origin rpy="0 0.09 0" xyz="0.0375 0.0005 0.0437"/>
-   <parent link="head_link"/>
-   <child link="jaw_link"/>
   </joint>
   <joint name="skull_joint" type="fixed">
@@ -92,3 +76,22 @@
   </joint>
 </xacro:macro>
+<xacro:macro name="head_jaw" params="covers">
+  <link name="jaw_link">
+    <visual>
+      <geometry>
+        <mesh filename="package://inmoov_meshes/meshes/jaw.stl" scale="0.001 0.001 0.001"/>
+      </geometry>
+      <origin rpy="0 0 0" xyz="0 0 0"/>
+      <xacro:cover_color/>
+    </visual>
+    <xacro:jaw_inertial/>
+  </link>
+  <joint name="head_jaw_joint" type="revolute">
+   <axis xyz="0 1 0"/>
+   <limit effort="1000.0" lower="${jaw_joint_lower}" upper="${jaw_joint_upper}" velocity="${jaw_joint_velocity}" />
+   <origin rpy="0 0.09 0" xyz="0.0375 0.0005 0.0437"/>
+   <parent link="head_link"/>
+   <child link="jaw_link"/>
+  </joint>
+</xacro:macro>
 </robot>

Commit message: add eye control to simulated robot, remove redundant "dynamixel-controllers" package
* right eye cannot be oriented horizontally currently

File: src/inmoov_description/robots/inmoov_head_control.urdf.xacro (robot description, xacro)
@@ -74,10 +74,9 @@
   </joint>
   <xacro:head covers="yes" />
-  <xacro:face covers="yes" />
-  <joint name="face_joint" type="fixed">
+  <!--<joint name="face_joint" type="fixed">
     <origin rpy="0 0 0" xyz="0.0637 0 0.079"/>
     <parent link="skull_link"/>
     <child link="face_link"/>
-  </joint>
+  </joint>-->
   <xacro:arm side="r" flip="1" covers="yes" />
   <joint name="r_shoulder_out_joint" type="revolute">

File: src/inmoov_description/urdf/asmFace.urdf.xacro (robot description, xacro)
@@ -1,50 +1,63 @@
 <?xml version="1.0"?>
-<robot name="inmoov" xmlns:xacro="http://ros.org/wiki/xacro">
-<xacro:include filename="$(find inmoov_description)/urdf/asmEye.urdf.xacro" />
-<xacro:macro name="face" params="covers">
-  <link name="face_link">
-    <visual>
-      <geometry>
-        <mesh filename="package://inmoov_meshes/meshes/face.stl" scale="0.001 0.001 0.001"/>
-      </geometry>
+<robot name="inmoov"
+  xmlns:xacro="http://ros.org/wiki/xacro">
+  <xacro:include filename="$(find inmoov_description)/urdf/asmEye.urdf.xacro" />
+  <xacro:macro name="face" params="covers">
+    <link name="face_link">
+      <visual>
+        <geometry>
+          <mesh filename="package://inmoov_meshes/meshes/face.stl" scale="0.001 0.001 0.001"/>
+        </geometry>
+        <origin rpy="0 0 0" xyz="0 0 0"/>
+        <xacro:cover_color/>
+      </visual>
+      <xacro:face_inertial/>
+    </link>
+    <joint name="eyes_shift_vertical_joint" type="revolute">
+      <axis xyz="0 1 0"/>
+      <limit effort="1000.0" lower="${eyes_tilt_joint_lower}" upper="${eyes_tilt_joint_upper}" velocity="${eyes_tilt_joint_velocity}" />
       <origin rpy="0 0 0" xyz="0 0 0"/>
-      <xacro:cover_color/>
-    </visual>
-    <xacro:face_inertial/>
-  </link>
-  <joint name="eyes_tilt_joint" type="revolute">
-   <axis xyz="0 1 0"/>
-   <limit effort="1000.0" lower="${eyes_tilt_joint_lower}" upper="${eyes_tilt_joint_upper}" velocity="${eyes_tilt_joint_velocity}" />
-   <origin rpy="0 0 0" xyz="0 0 0"/>
-   <parent link="face_link"/>
-   <child link="eyesupport_link"/>
-  </joint>
-  <link name="eyesupport_link">
-    <visual>
-      <geometry>
-        <mesh filename="package://inmoov_meshes/meshes/eyesupport.stl" scale="0.001 0.001 0.001"/>
-      </geometry>
+      <parent link="face_link"/>
+      <child link="eyesupport_link"/>
+    </joint>
+    <!--<joint name="eyes_shift_horizontal_joint" type="revolute">
+      <axis xyz="1 0 0"/>
+      <limit effort="1000.0" lower="${eyes_pan_joint_lower}" upper="${eyes_pan_joint_upper}" velocity="${eyes_pan_joint_velocity}" />
       <origin rpy="0 0 0" xyz="0 0 0"/>
-      <xacro:frame_color/>
-    </visual>
-    <xacro:eyesupport_inertial/>
-  </link>
-<xacro:asmEye side="r"/>
-  <joint name="eyes_pan_joint" type="revolute">
-   <axis xyz="0 0 1"/>
-    <limit effort="1000.0" lower="${eyes_pan_joint_lower}" upper="${eyes_pan_joint_upper}" velocity="${eyes_pan_joint_velocity}" />
-   <origin rpy="0 0 0" xyz="0 0.033 -0.0036"/>
-   <parent link="eyesupport_link"/>
-   <child link="r_eyesupport_link"/>
-  </joint>
-<xacro:asmEye side="l" />
-  <joint name="l_eye_pan_joint" type="revolute">
-   <axis xyz="0 0 1"/>
-   <limit effort="1000.0" lower="${eyes_pan_joint_lower}" upper="${eyes_pan_joint_upper}" velocity="${eyes_pan_joint_velocity}" />
-   <mimic joint="eyes_pan_joint" multiplier="1" offset="0"/>
-   <origin rpy="0 0 0" xyz="0 -0.033 -0.0036"/>
-   <parent link="eyesupport_link"/>
-   <child link="l_eyesupport_link"/>
-  </joint>
-</xacro:macro>
+      <parent link="face_link"/>
+      <child link="eyesupport_link"/>
+    </joint>-->
+    <link name="eyesupport_link">
+      <visual>
+        <geometry>
+          <mesh filename="package://inmoov_meshes/meshes/eyesupport.stl" scale="0.001 0.001 0.001"/>
+        </geometry>
+        <origin rpy="0 0 0" xyz="0 0 0"/>
+        <xacro:frame_color/>
+      </visual>
+      <xacro:eyesupport_inertial/>
+    </link>
+    <xacro:asmEye side="r"/>
+    <joint name="eyes_shift_horizontal_joint" type="revolute">
+      <axis xyz="0 0 1"/>
+      <limit effort="1000.0" lower="${eyes_pan_joint_lower}" upper="${eyes_pan_joint_upper}" velocity="${eyes_pan_joint_velocity}" />
+      <origin rpy="0 0 0" xyz="0 0.033 -0.0036"/>
+      <parent link="eyesupport_link"/>
+      <child link="r_eyesupport_link"/>
+    </joint>
+    <!--<joint name="r_eye_shift_horizontal_joint" type="fixed">
+      <origin rpy="0 0 0" xyz="0 0.033 -0.0036"/>
+      <parent link="eyesupport_link"/>
+      <child link="r_eyesupport_link"/>
+    </joint>-->
+    <xacro:asmEye side="l" />
+    <joint name="l_eye_shift_horizontal_joint" type="revolute">
+      <axis xyz="0 0 1"/>
+      <limit effort="1000.0" lower="${eyes_pan_joint_lower}" upper="${eyes_pan_joint_upper}" velocity="${eyes_pan_joint_velocity}" />
+      <mimic joint="eyes_shift_horizontal_joint" multiplier="1" offset="0"/>
+      <origin rpy="0 0 0" xyz="0 -0.033 -0.0036"/>
+      <parent link="eyesupport_link"/>
+      <child link="l_eyesupport_link"/>
+    </joint>
+  </xacro:macro>
 </robot>
