Commit message: Robot launch fixes

File: src/inmoov_description/robots/inmoov.urdf_old.xacro (robot description, xacro)
@@ -15,8 +15,20 @@
 <!-- Import ros2_control description -->
   <xacro:include filename="head.ros2_control.xacro" />
-  <link name="world"/>
+  <!--<xacro:rrbot parent="world" prefix="$(arg prefix)">
+    <origin xyz="0 0 0" rpy="0 0 0" />
+  </xacro:rrbot>-->
+  <xacro:arg name="fake_sensor_commands" default="true" />
+  <xacro:arg name="use_fake_hardware" default="true" />
+  <!--
+  -->
+  <xacro:arg name="prefix" default="" />
+  <xacro:arg name="slowdown" default="2.0" />
+  <link name="world">
+  </link>
   <joint name="fixed" type="fixed">
     <parent link="world"/>
     <child link="base_link"/>
+    <origin xyz="0 0 0" rpy="0 0 0" />
+    <axis xyz="1 0 0"/>
   </joint>
   <link name="base_link">
@@ -26,6 +38,8 @@
       </geometry>
       <origin rpy="0 0 0" xyz="0 0 0.055"/>
+      <axis xyz="1 0 0"/>
       <xacro:base_color/>
     </visual>
+    <axis xyz="1 0 0"/>
   </link>
   <joint name="base_to_pedestal_link" type="fixed">
@@ -113,4 +127,7 @@
    <child link="l_hand_link"/>
   </joint>
-  <xacro:robot_head name="RobotHead" prefix="" />
+  <xacro:robot_head name="RobotHead" prefix=""
+    use_fake_hardware="$(arg use_fake_hardware)"
+    fake_sensor_commands="$(arg fake_sensor_commands)"
+    slowdown="$(arg slowdown)"/>
 </robot>
