Commit message: Fixed simulation after joelryt-merge

File: src/inmoov_description/robots/head.ros2_control_old.xacro (robot description, xacro)
@@ -70,4 +70,60 @@
         <state_interface name="velocity"/>
       </joint>
+      <joint name="r_shoulder_lift_joint">
+        <command_interface name="position">
+          <param name="min">-1</param>
+          <param name="max">1</param>
+        </command_interface>
+        <state_interface name="position"/>
+        <state_interface name="velocity"/>
+      </joint>
+      <joint name="r_shoulder_out_joint">
+        <command_interface name="position">
+          <param name="min">-1</param>
+          <param name="max">1</param>
+        </command_interface>
+        <state_interface name="position"/>
+        <state_interface name="velocity"/>
+      </joint>
+      <joint name="r_thumb_joint">
+        <command_interface name="position">
+          <param name="min">-1</param>
+          <param name="max">1</param>
+        </command_interface>
+        <state_interface name="position"/>
+        <state_interface name="velocity"/>
+      </joint>
+      <joint name="r_index1_joint">
+        <command_interface name="position">
+          <param name="min">-1</param>
+          <param name="max">1</param>
+        </command_interface>
+        <state_interface name="position"/>
+        <state_interface name="velocity"/>
+      </joint>
+      <joint name="r_middle1_joint">
+        <command_interface name="position">
+          <param name="min">-1</param>
+          <param name="max">1</param>
+        </command_interface>
+        <state_interface name="position"/>
+        <state_interface name="velocity"/>
+      </joint>
+      <joint name="r_ring_joint">
+        <command_interface name="position">
+          <param name="min">-1</param>
+          <param name="max">1</param>
+        </command_interface>
+        <state_interface name="position"/>
+        <state_interface name="velocity"/>
+      </joint>
+      <joint name="r_pinky_joint">
+        <command_interface name="position">
+          <param name="min">-1</param>
+          <param name="max">1</param>
+        </command_interface>
+        <state_interface name="position"/>
+        <state_interface name="velocity"/>
+      </joint>
     </ros2_control>
   </xacro:macro>

File: src/inmoov_description/robots/inmoov.urdf.xacro (robot description, xacro)
@@ -14,10 +14,10 @@
   <xacro:include filename="$(find inmoov_description)/urdf/asmHand.urdf.xacro" />
 <!-- Import ros2_control description -->
-  <xacro:include filename="head.ros2_control.xacro" />
+  <xacro:include filename="head.ros2_control_old.xacro" />
   <!--<xacro:rrbot parent="world" prefix="$(arg prefix)">
     <origin xyz="0 0 0" rpy="0 0 0" />
   </xacro:rrbot>-->
-  <xacro:arg name="fake_sensor_commands" default="false" />
-  <xacro:arg name="use_fake_hardware" default="false" />
+  <xacro:arg name="fake_sensor_commands" default="true" />
+  <xacro:arg name="use_fake_hardware" default="true" />
   <!--
   -->
