Commit message: Update joint config, add dynamixel comm to robot_hardware

File: src/inmoov_description/robots/head.ros2_control.xacro (robot description, xacro)
@@ -17,4 +17,28 @@
         <state_interface name="velocity"/>
       </joint>
+      <joint name="head_tilt_right_joint">
+        <command_interface name="position">
+          <param name="min">-1</param>
+          <param name="max">1</param>
+        </command_interface>
+        <state_interface name="position"/>
+        <state_interface name="velocity"/>
+      </joint>
+      <joint name="head_tilt_left_joint">
+        <command_interface name="position">
+          <param name="min">-1</param>
+          <param name="max">1</param>
+        </command_interface>
+        <state_interface name="position"/>
+        <state_interface name="velocity"/>
+      </joint>
+      <joint name="head_tilt_vertical_joint">
+        <command_interface name="position">
+          <param name="min">-1</param>
+          <param name="max">1</param>
+        </command_interface>
+        <state_interface name="position"/>
+        <state_interface name="velocity"/>
+      </joint>
     </ros2_control>
   </xacro:macro>

Commit message: Add rest of head joints

File: src/inmoov_description/robots/head.ros2_control.xacro (robot description, xacro)
@@ -7,4 +7,12 @@
         <param name="dynamixel_info">config/dynamixel.yaml</param>
       </hardware>
+      <joint name="head_jaw_joint">
+        <command_interface name="position">
+          <param name="min">-1</param>
+          <param name="max">1</param>
+        </command_interface>
+        <state_interface name="position"/>
+        <state_interface name="velocity"/>
+      </joint>
       <joint name="head_pan_joint">
         <command_interface name="position">

Commit message: Add joint controllers, fix robot hardware bugs

File: src/inmoov_description/robots/head.ros2_control.xacro (robot description, xacro)
@@ -1,5 +1,5 @@
 <?xml version="1.0"?>
 <robot xmlns:xacro="http://www.ros.org/wiki/xacro">
-  <xacro:macro name="robot_head_pan" params="name prefix">
+  <xacro:macro name="robot_head" params="name prefix">
     <ros2_control name="${name}" type="system">
       <hardware>
@@ -41,4 +41,20 @@
       <joint name="head_tilt_vertical_joint">
         <command_interface name="position">
+          <param name="min">-1.5</param>
+          <param name="max">0</param>
+        </command_interface>
+        <state_interface name="position"/>
+        <state_interface name="velocity"/>
+      </joint>
+      <joint name="eyes_shift_horizontal_joint">
+        <command_interface name="position">
+          <param name="min">-1</param>
+          <param name="max">1</param>
+        </command_interface>
+        <state_interface name="position"/>
+        <state_interface name="velocity"/>
+      </joint>
+      <joint name="eyes_shift_vertical_joint">
+        <command_interface name="position">
           <param name="min">-1</param>
           <param name="max">1</param>

File: src/inmoov_description/robots/inmoov.urdf.xacro (robot description, xacro)
@@ -112,4 +112,4 @@
    <child link="l_hand_link"/>
   </joint>
-  <xacro:robot_head_pan name="RobotHeadPan" prefix="" />
+  <xacro:robot_head name="RobotHead" prefix="" />
 </robot>

Commit message: WIP to fix sim. Attemt to rewrite based on ros2_control_demo examples, joint states seem non-nan now and nan err fixed but sim still broken

File: src/inmoov_description/robots/head.ros2_control.xacro (robot description, xacro)
@@ -1,9 +1,16 @@
 <?xml version="1.0"?>
 <robot xmlns:xacro="http://www.ros.org/wiki/xacro">
-  <xacro:macro name="robot_head" params="name prefix">
+  <xacro:macro name="robot_head" params="name prefix use_fake_hardware:=^|true fake_sensor_commands:=^|false slowdown:=2.0">
     <ros2_control name="${name}" type="system">
       <hardware>
+        <xacro:if value="${use_fake_hardware}">
+          <plugin>fake_components/GenericSystem</plugin>
+          <param name="fake_sensor_commands">${fake_sensor_commands}</param>
+          <param name="state_following_offset">0.0</param>
+        </xacro:if>
+        <xacro:unless value="${use_fake_hardware}">
         <plugin>robot_hardware/RobotHardware</plugin>
         <param name="dynamixel_info">config/dynamixel.yaml</param>
+        </xacro:unless>
       </hardware>
       <joint name="head_jaw_joint">

File: src/inmoov_description/robots/inmoov.urdf.xacro (robot description, xacro)
@@ -15,8 +15,20 @@
 <!-- Import ros2_control description -->
   <xacro:include filename="head.ros2_control.xacro" />
-  <link name="world"/>
+  <!--<xacro:rrbot parent="world" prefix="$(arg prefix)">
+    <origin xyz="0 0 0" rpy="0 0 0" />
+  </xacro:rrbot>-->
+  <xacro:arg name="fake_sensor_commands" default="true" />
+  <xacro:arg name="use_fake_hardware" default="true" />
+  <!--
+  -->
+  <xacro:arg name="prefix" default="" />
+  <xacro:arg name="slowdown" default="2.0" />
+  <link name="world">
+  </link>
   <joint name="fixed" type="fixed">
     <parent link="world"/>
     <child link="base_link"/>
+    <origin xyz="0 0 0" rpy="0 0 0" />
+    <axis xyz="1 0 0"/>
   </joint>
   <link name="base_link">
@@ -26,6 +38,8 @@
       </geometry>
       <origin rpy="0 0 0" xyz="0 0 0.055"/>
+      <axis xyz="1 0 0"/>
       <xacro:base_color/>
     </visual>
+    <axis xyz="1 0 0"/>
   </link>
   <joint name="base_to_pedestal_link" type="fixed">
@@ -113,4 +127,9 @@
    <child link="l_hand_link"/>
   </joint>
-  <xacro:robot_head name="RobotHead" prefix="" />
+  <!--
+  -->
+  <xacro:robot_head name="RobotHead" prefix=""
+    use_fake_hardware="$(arg use_fake_hardware)"
+    fake_sensor_commands="$(arg fake_sensor_commands)"
+    slowdown="$(arg slowdown)"/>
 </robot>

Commit message: Working base for hand movement

File: src/inmoov_description/robots/head.ros2_control.xacro (robot description, xacro)
@@ -70,4 +70,60 @@
         <state_interface name="velocity"/>
       </joint>
+      <joint name="r_shoulder_lift_joint">
+        <command_interface name="position">
+          <param name="min">-1</param>
+          <param name="max">1</param>
+        </command_interface>
+        <state_interface name="position"/>
+        <state_interface name="velocity"/>
+      </joint>
+      <joint name="r_shoulder_out_joint">
+        <command_interface name="position">
+          <param name="min">-1</param>
+          <param name="max">1</param>
+        </command_interface>
+        <state_interface name="position"/>
+        <state_interface name="velocity"/>
+      </joint>
+      <joint name="r_thumb_joint">
+        <command_interface name="position">
+          <param name="min">-1</param>
+          <param name="max">1</param>
+        </command_interface>
+        <state_interface name="position"/>
+        <state_interface name="velocity"/>
+      </joint>
+      <joint name="r_index1_joint">
+        <command_interface name="position">
+          <param name="min">-1</param>
+          <param name="max">1</param>
+        </command_interface>
+        <state_interface name="position"/>
+        <state_interface name="velocity"/>
+      </joint>
+      <joint name="r_middle1_joint">
+        <command_interface name="position">
+          <param name="min">-1</param>
+          <param name="max">1</param>
+        </command_interface>
+        <state_interface name="position"/>
+        <state_interface name="velocity"/>
+      </joint>
+      <joint name="r_ring_joint">
+        <command_interface name="position">
+          <param name="min">-1</param>
+          <param name="max">1</param>
+        </command_interface>
+        <state_interface name="position"/>
+        <state_interface name="velocity"/>
+      </joint>
+      <joint name="r_pinky_joint">
+        <command_interface name="position">
+          <param name="min">-1</param>
+          <param name="max">1</param>
+        </command_interface>
+        <state_interface name="position"/>
+        <state_interface name="velocity"/>
+      </joint>
     </ros2_control>
   </xacro:macro>

Commit message: Dynamixel servo config file path can now be given as argument for robot.launch.py. WIP to get physical arm+hand and head running separately without errors.

File: src/inmoov_description/robots/head.ros2_control.xacro (robot description, xacro)
@@ -1,9 +1,10 @@
 <?xml version="1.0"?>
 <robot xmlns:xacro="http://www.ros.org/wiki/xacro">
-  <xacro:macro name="robot_head" params="name prefix">
+  <xacro:macro name="robot_head" params="name prefix dynamixel_config_file">
     <ros2_control name="${name}" type="system">
       <hardware>
         <plugin>robot_hardware/RobotHardware</plugin>
-        <param name="dynamixel_info">config/dynamixel.yaml</param>
+        <!--<param name="dynamixel_info">config/dynamixel.yaml</param>-->
+        <param name="dynamixel_info">${dynamixel_config_file}</param>
       </hardware>
       <joint name="head_jaw_joint">

File: src/inmoov_description/robots/head.ros2_control_old.xacro (robot description, xacro)
@@ -1,5 +1,5 @@
 <?xml version="1.0"?>
 <robot xmlns:xacro="http://www.ros.org/wiki/xacro">
-  <xacro:macro name="robot_head" params="name prefix use_fake_hardware:=^|true fake_sensor_commands:=^|false slowdown:=2.0">
+  <xacro:macro name="robot_head" params="name prefix use_fake_hardware:=^|true fake_sensor_commands:=^|false slowdown:=2.0 dynamixel_config_file">
     <ros2_control name="${name}" type="system">
       <hardware>
@@ -11,5 +11,6 @@
         <xacro:unless value="${use_fake_hardware}">
         <plugin>robot_hardware/RobotHardware</plugin>
-        <param name="dynamixel_info">config/dynamixel.yaml</param>
+        <!--<param name="dynamixel_info">config/dynamixel.yaml</param>-->
+        <param name="dynamixel_info">${dynamixel_config_file}</param>
         </xacro:unless>
       </hardware>

File: src/inmoov_description/robots/inmoov.urdf.xacro (robot description, xacro)
@@ -24,4 +24,5 @@
   <xacro:arg name="prefix" default="" />
   <xacro:arg name="slowdown" default="2.0" />
+  <xacro:arg name="dynamixel_config_file" default="NOT_SET_2" />
   <link name="world">
   </link>
@@ -130,4 +131,5 @@
     use_fake_hardware="$(arg use_fake_hardware)"
     fake_sensor_commands="$(arg fake_sensor_commands)"
-    slowdown="$(arg slowdown)"/>
+    slowdown="$(arg slowdown)"
+    dynamixel_config_file="$(arg dynamixel_config_file)"/>
 </robot>

Commit message: Removed "old" from the names of head.ros2_control_old.xacro and inmoov.urdf_old.xacro and deleted the corresponding files that had no "old" in their names.

File: src/inmoov_description/robots/head.ros2_control.xacro (robot description, xacro)
@@ -1,10 +1,17 @@
 <?xml version="1.0"?>
 <robot xmlns:xacro="http://www.ros.org/wiki/xacro">
-  <xacro:macro name="robot_head" params="name prefix dynamixel_config_file">
+  <xacro:macro name="robot_head" params="name prefix use_fake_hardware:=^|true fake_sensor_commands:=^|false slowdown:=2.0 dynamixel_config_file">
     <ros2_control name="${name}" type="system">
       <hardware>
+        <xacro:if value="${use_fake_hardware}">
+          <plugin>fake_components/GenericSystem</plugin>
+          <param name="fake_sensor_commands">${fake_sensor_commands}</param>
+          <param name="state_following_offset">0.0</param>
+        </xacro:if>
+        <xacro:unless value="${use_fake_hardware}">
         <plugin>robot_hardware/RobotHardware</plugin>
         <!--<param name="dynamixel_info">config/dynamixel.yaml</param>-->
         <param name="dynamixel_info">${dynamixel_config_file}</param>
+        </xacro:unless>
       </hardware>
       <joint name="head_jaw_joint">

File: src/inmoov_description/robots/inmoov.urdf.xacro (robot description, xacro)
@@ -14,5 +14,5 @@
   <xacro:include filename="$(find inmoov_description)/urdf/asmHand.urdf.xacro" />
 <!-- Import ros2_control description -->
-  <xacro:include filename="head.ros2_control_old.xacro" />
+  <xacro:include filename="head.ros2_control.xacro" />
   <!--<xacro:rrbot parent="world" prefix="$(arg prefix)">
     <origin xyz="0 0 0" rpy="0 0 0" />
