Commit message: WIP: fixed some joints to make robot partially show at sim

File: src/inmoov_description/robots/inmoov.urdf.xacro (robot description, xacro)
@@ -73,5 +73,7 @@
   </joint>
   <xacro:torso covers="yes" />
-  <joint name="head_roll_joint" type="revolute">
+<!-- Test what happens when fixing also this joint to create joint chain
+  <joint name="head_roll_joint" type="revolute">-->
+  <joint name="head_roll_joint" type="fixed">
    <axis xyz="1 0 0"/>
    <limit effort="1000.0" lower="${head_roll_joint_lower}" upper="${head_roll_joint_upper}" velocity="${head_roll_joint_velocity}" />
@@ -80,5 +82,7 @@
    <child link="head_tilt_link"/>
   </joint>
-  <joint name="head_tilt_joint" type="revolute">
+  <!-- Test what happens when fixing joint
+    <joint name="head_tilt_joint" type="revolute">-->
+  <joint name="head_tilt_joint" type="fixed">
    <axis xyz="0 1 0"/>
    <limit effort="1000.0" lower="${head_tilt_joint_lower}" upper="${head_tilt_joint_upper}" velocity="${head_tilt_joint_velocity}" />
@@ -127,6 +131,4 @@
    <child link="l_hand_link"/>
   </joint>
-  <!--
-  -->
   <xacro:robot_head name="RobotHead" prefix=""
     use_fake_hardware="$(arg use_fake_hardware)"

File: src/inmoov_description/urdf/asmTorso.urdf.xacro (robot description, xacro)
@@ -82,5 +82,7 @@
     <xacro:chest_inertial/>
   </link>
-  <joint name="waist_pan_joint" type="revolute">
+  <!--Fixing links until getting head to show
+  <joint name="waist_pan_joint" type="revolute">-->
+  <joint name="waist_pan_joint" type="fixed">
    <axis xyz="0 0 1"/>
    <limit effort="1000.0" lower="${waist_pan_joint_lower}" upper="${waist_pan_joint_upper}" velocity="${waist_pan_joint_velocity}" />
@@ -94,5 +96,7 @@
     <child link="disk_link"/>
   </joint>
-  <joint name="waist_roll_joint" type="revolute">
+  <!--Fixing links until getting head to show
+  <joint name="waist_roll_joint" type="revolute">-->
+  <joint name="waist_roll_joint" type="fixed">
    <axis xyz="1 0 0"/>
    <limit effort="1000.0" lower="${waist_roll_joint_lower}" upper="${waist_roll_joint_upper}" velocity="${waist_roll_joint_velocity}" />

Commit message: Turn previous fixed joints back to revolute

File: src/inmoov_description/robots/inmoov.urdf.xacro (robot description, xacro)
@@ -73,7 +73,5 @@
   </joint>
   <xacro:torso covers="yes" />
-<!-- Test what happens when fixing also this joint to create joint chain
-  <joint name="head_roll_joint" type="revolute">-->
-  <joint name="head_roll_joint" type="fixed">
+  <joint name="head_roll_joint" type="revolute">
    <axis xyz="1 0 0"/>
    <limit effort="1000.0" lower="${head_roll_joint_lower}" upper="${head_roll_joint_upper}" velocity="${head_roll_joint_velocity}" />
@@ -82,7 +80,5 @@
    <child link="head_tilt_link"/>
   </joint>
-  <!-- Test what happens when fixing joint
-    <joint name="head_tilt_joint" type="revolute">-->
-  <joint name="head_tilt_joint" type="fixed">
+  <joint name="head_tilt_joint" type="revolute">
    <axis xyz="0 1 0"/>
    <limit effort="1000.0" lower="${head_tilt_joint_lower}" upper="${head_tilt_joint_upper}" velocity="${head_tilt_joint_velocity}" />

File: src/inmoov_description/urdf/asmTorso.urdf.xacro (robot description, xacro)
@@ -82,7 +82,5 @@
     <xacro:chest_inertial/>
   </link>
-  <!--Fixing links until getting head to show
-  <joint name="waist_pan_joint" type="revolute">-->
-  <joint name="waist_pan_joint" type="fixed">
+  <joint name="waist_pan_joint" type="revolute">
    <axis xyz="0 0 1"/>
    <limit effort="1000.0" lower="${waist_pan_joint_lower}" upper="${waist_pan_joint_upper}" velocity="${waist_pan_joint_velocity}" />
@@ -96,7 +94,5 @@
     <child link="disk_link"/>
   </joint>
-  <!--Fixing links until getting head to show
-  <joint name="waist_roll_joint" type="revolute">-->
-  <joint name="waist_roll_joint" type="fixed">
+  <joint name="waist_roll_joint" type="revolute">
    <axis xyz="1 0 0"/>
    <limit effort="1000.0" lower="${waist_roll_joint_lower}" upper="${waist_roll_joint_upper}" velocity="${waist_roll_joint_velocity}" />

Commit message: Changed the word "head" to "robot" in some files that include also arm and hand and not only head. Deleted the unused file head_old.yaml.

File: src/inmoov_description/robots/inmoov.urdf.xacro (robot description, xacro)
@@ -14,5 +14,5 @@
   <xacro:include filename="$(find inmoov_description)/urdf/asmHand.urdf.xacro" />
 <!-- Import ros2_control description -->
-  <xacro:include filename="head.ros2_control.xacro" />
+  <xacro:include filename="robot.ros2_control.xacro" />
   <!--<xacro:rrbot parent="world" prefix="$(arg prefix)">
     <origin xyz="0 0 0" rpy="0 0 0" />
@@ -128,5 +128,5 @@
    <child link="l_hand_link"/>
   </joint>
-  <xacro:robot_head name="RobotHead" prefix=""
+  <xacro:robot name="Robot" prefix=""
     use_fake_hardware="$(arg use_fake_hardware)"
     fake_sensor_commands="$(arg fake_sensor_commands)"

File: src/inmoov_description/robots/inmoov_eyes_control.urdf.xacro (robot description, xacro)
@@ -14,6 +14,6 @@
   <xacro:include filename="$(find inmoov_description)/urdf/asmHand.urdf.xacro" />
   <!-- Import ros2_control description -->
-  <xacro:include filename="head.ros2_control.xacro" />
+  <xacro:include filename="robot.ros2_control.xacro" />
   <xacro:face covers="yes" />
-  <xacro:robot_head name="RobotHead" prefix="" />
+  <xacro:robot name="Robot" prefix="" />
 </robot>

File: src/inmoov_description/robots/inmoov_head_control.urdf.xacro (robot description, xacro)
@@ -14,5 +14,5 @@
   <xacro:include filename="$(find inmoov_description)/urdf/asmHand.urdf.xacro" />
 <!-- Import ros2_control description -->
-  <xacro:include filename="head.ros2_control.xacro" />
+  <xacro:include filename="robot.ros2_control.xacro" />
   <link name="world"/>
   <joint name="fixed" type="fixed">
@@ -111,4 +111,4 @@
    <child link="l_hand_link"/>
   </joint>
-  <xacro:robot_head name="RobotHead" prefix="" />
+  <xacro:robot name="Robot" prefix="" />
 </robot>

File: src/inmoov_description/robots/inmoov_jaw_control.urdf.xacro (robot description, xacro)
@@ -14,6 +14,6 @@
   <xacro:include filename="$(find inmoov_description)/urdf/asmHand.urdf.xacro" />
   <!-- Import ros2_control description -->
-  <xacro:include filename="head.ros2_control.xacro" />
+  <xacro:include filename="robot.ros2_control.xacro" />
   <xacro:head_jaw covers="yes" />
-  <xacro:robot_head name="RobotHead" prefix="" />
+  <xacro:robot name="Robot" prefix="" />
 </robot>

File: src/inmoov_description/robots/robot.ros2_control.xacro (robot description, xacro)
@@ -1,5 +1,5 @@
 <?xml version="1.0"?>
 <robot xmlns:xacro="http://www.ros.org/wiki/xacro">
-  <xacro:macro name="robot_head" params="name prefix use_fake_hardware:=^|true fake_sensor_commands:=^|false slowdown:=2.0 dynamixel_config_file">
+  <xacro:macro name="robot" params="name prefix use_fake_hardware:=^|true fake_sensor_commands:=^|false slowdown:=2.0 dynamixel_config_file">
     <ros2_control name="${name}" type="system">
       <hardware>
@@ -11,5 +11,4 @@
         <xacro:unless value="${use_fake_hardware}">
         <plugin>robot_hardware/RobotHardware</plugin>
-        <!--<param name="dynamixel_info">config/dynamixel.yaml</param>-->
         <param name="dynamixel_info">${dynamixel_config_file}</param>
         </xacro:unless>

Commit message: humble hardware version test

File: src/inmoov_description/robots/inmoov.urdf.xacro (robot description, xacro)
@@ -18,11 +18,11 @@
     <origin xyz="0 0 0" rpy="0 0 0" />
   </xacro:rrbot>-->
+    <!--
   <xacro:arg name="fake_sensor_commands" default="true" />
   <xacro:arg name="use_fake_hardware" default="true" />
-  <!--
-  -->
   <xacro:arg name="prefix" default="" />
   <xacro:arg name="slowdown" default="2.0" />
   <xacro:arg name="dynamixel_config_file" default="NOT_SET_2" />
+  -->
   <link name="world">
   </link>
@@ -128,8 +128,4 @@
    <child link="l_hand_link"/>
   </joint>
-  <xacro:robot name="Robot" prefix=""
-    use_fake_hardware="$(arg use_fake_hardware)"
-    fake_sensor_commands="$(arg fake_sensor_commands)"
-    slowdown="$(arg slowdown)"
-    dynamixel_config_file="$(arg dynamixel_config_file)"/>
+  <xacro:robot name="Robot"/>
 </robot>

File: src/inmoov_description/robots/robot.ros2_control.xacro (robot description, xacro)
@@ -1,166 +1,123 @@
 <?xml version="1.0"?>
 <robot xmlns:xacro="http://www.ros.org/wiki/xacro">
-  <xacro:macro name="robot" params="name prefix use_fake_hardware:=^|true fake_sensor_commands:=^|false slowdown:=2.0 dynamixel_config_file">
+  <xacro:macro name="robot" params="name">
     <ros2_control name="${name}" type="system">
       <hardware>
-        <xacro:if value="${use_fake_hardware}">
-          <plugin>fake_components/GenericSystem</plugin>
-          <param name="fake_sensor_commands">${fake_sensor_commands}</param>
-          <param name="state_following_offset">0.0</param>
-        </xacro:if>
-        <xacro:unless value="${use_fake_hardware}">
-        <plugin>robot_hardware/RobotHardware</plugin>
-        <param name="dynamixel_info">${dynamixel_config_file}</param>
-        </xacro:unless>
+        <plugin>dynamixel_hardware/DynamixelHardware</plugin>
+        <param name="usb_port">/dev/ttyUSB0</param>
+        <param name="baud_rate">1000000</param>
+        <param name="use_dummy">true</param>
       </hardware>
       <joint name="head_jaw_joint">
-        <command_interface name="position">
-          <param name="min">-1</param>
-          <param name="max">1</param>
-        </command_interface>
+        <command_interface name="position"/>
+         <param name="id">11</param>
         <state_interface name="position"/>
         <state_interface name="velocity"/>
       </joint>
       <joint name="head_pan_joint">
-        <command_interface name="position">
-          <param name="min">-1</param>
-          <param name="max">1</param>
-        </command_interface>
+        <command_interface name="position"/>
+          <param name="id">12</param>
         <state_interface name="position"/>
         <state_interface name="velocity"/>
       </joint>
       <joint name="head_tilt_right_joint">
-        <command_interface name="position">
-          <param name="min">-1</param>
-          <param name="max">1</param>
-        </command_interface>
+        <command_interface name="position"/>
+          <param name="id">13</param>
         <state_interface name="position"/>
         <state_interface name="velocity"/>
       </joint>
       <joint name="head_tilt_left_joint">
-        <command_interface name="position">
-          <param name="min">-1</param>
-          <param name="max">1</param>
-        </command_interface>
+        <command_interface name="position"/>
+          <param name="id">14</param>
         <state_interface name="position"/>
         <state_interface name="velocity"/>
       </joint>
       <joint name="head_tilt_vertical_joint">
-        <command_interface name="position">
-          <param name="min">-1.5</param>
-          <param name="max">0</param>
-        </command_interface>
+        <command_interface name="position"/>
+        <param name="id">15</param>
         <state_interface name="position"/>
         <state_interface name="velocity"/>
       </joint>
       <joint name="eyes_shift_horizontal_joint">
-        <command_interface name="position">
-          <param name="min">-1</param>
-          <param name="max">1</param>
-        </command_interface>
+        <command_interface name="position"/>
+          <param name="id">16</param>
         <state_interface name="position"/>
         <state_interface name="velocity"/>
       </joint>
       <joint name="eyes_shift_vertical_joint">
-        <command_interface name="position">
-          <param name="min">-1</param>
-          <param name="max">1</param>
-        </command_interface>
+        <command_interface name="position"/>
+          <param name="id">17</param>
         <state_interface name="position"/>
         <state_interface name="velocity"/>
       </joint>
       <joint name="r_shoulder_lift_joint">
-        <command_interface name="position">
-          <param name="min">-1</param>
-          <param name="max">1</param>
-        </command_interface>
+        <command_interface name="position"/>
+          <param name="id">18</param>
         <state_interface name="position"/>
         <state_interface name="velocity"/>
       </joint>
       <joint name="r_shoulder_out_joint">
-        <command_interface name="position">
-          <param name="min">-1</param>
-          <param name="max">1</param>
-        </command_interface>
+        <command_interface name="position"/>
+          <param name="id">19</param>
         <state_interface name="position"/>
         <state_interface name="velocity"/>
       </joint>
       <joint name="r_thumb_joint">
-        <command_interface name="position">
-          <param name="min">-1</param>
-          <param name="max">1</param>
-        </command_interface>
+        <command_interface name="position"/>
+          <param name="id">20</param>
         <state_interface name="position"/>
         <state_interface name="velocity"/>
       </joint>
       <joint name="r_index1_joint">
-        <command_interface name="position">
-          <param name="min">-1</param>
-          <param name="max">1</param>
-        </command_interface>
+        <command_interface name="position"/>
+          <param name="id">21</param>
         <state_interface name="position"/>
         <state_interface name="velocity"/>
       </joint>
       <joint name="r_middle1_joint">
-        <command_interface name="position">
-          <param name="min">-1</param>
-          <param name="max">1</param>
-        </command_interface>
+        <command_interface name="position"/>
+          <param name="id">22</param>
         <state_interface name="position"/>
         <state_interface name="velocity"/>
       </joint>
       <joint name="r_ring_joint">
-        <command_interface name="position">
-          <param name="min">-1</param>
-          <param name="max">1</param>
-        </command_interface>
+        <command_interface name="position"/>
+          <param name="id">23</param>
         <state_interface name="position"/>
         <state_interface name="velocity"/>
       </joint>
       <joint name="r_pinky_joint">
-        <command_interface name="position">
-          <param name="min">-1</param>
-          <param name="max">1</param>
-        </command_interface>
+        <command_interface name="position"/>
+          <param name="id">24</param>
         <state_interface name="position"/>
         <state_interface name="velocity"/>
       </joint>
       <joint name="l_thumb_joint">
-        <command_interface name="position">
-          <param name="min">-1</param>
-          <param name="max">1</param>
-        </command_interface>
+        <command_interface name="position"/>
+          <param name="id">25</param>
         <state_interface name="position"/>
         <state_interface name="velocity"/>
       </joint>
       <joint name="l_index1_joint">
-        <command_interface name="position">
-          <param name="min">-1</param>
-          <param name="max">1</param>
-        </command_interface>
+        <command_interface name="position"/>
+          <param name="id">26</param>
         <state_interface name="position"/>
         <state_interface name="velocity"/>
       </joint>
       <joint name="l_middle1_joint">
-        <command_interface name="position">
-          <param name="min">-1</param>
-          <param name="max">1</param>
-        </command_interface>
+        <command_interface name="position"/>
+          <param name="id">27</param>
         <state_interface name="position"/>
         <state_interface name="velocity"/>
       </joint>
       <joint name="l_ring_joint">
-        <command_interface name="position">
-          <param name="min">-1</param>
-          <param name="max">1</param>
-        </command_interface>
+        <command_interface name="position"/>
+          <param name="id">28</param>
         <state_interface name="position"/>
         <state_interface name="velocity"/>
       </joint>
       <joint name="l_pinky_joint">
-        <command_interface name="position">
-          <param name="min">-1</param>
-          <param name="max">1</param>
-        </command_interface>
+        <command_interface name="position"/>
+          <param name="id">29</param>
         <state_interface name="position"/>
         <state_interface name="velocity"/>

File: src/inmoov_description/urdf/config.joints.urdf.xacro (robot description, xacro)
@@ -2,5 +2,5 @@
 <robot xmlns:xacro="http://ros.org/wiki/xacro">
   <xacro:property name="filename" value="$(find inmoov_description)/config/config.yaml"/>
-  <xacro:property name="c" value="${load_yaml(filename)}"/>
+  <xacro:property name="c" value="${xacro.load_yaml(filename)}"/>
   <!--xacro:property name="pi" value="3.1415926539"/-->
   <xacro:if value="${c['bringup']['angles'] == 'degrees'}">

Commit message: robot hardware ready to test

File: src/inmoov_description/robots/inmoov.urdf.xacro (robot description, xacro)
@@ -18,5 +18,4 @@
     <origin xyz="0 0 0" rpy="0 0 0" />
   </xacro:rrbot>-->
-    <!--
   <xacro:arg name="fake_sensor_commands" default="true" />
   <xacro:arg name="use_fake_hardware" default="true" />
@@ -24,5 +23,4 @@
   <xacro:arg name="slowdown" default="2.0" />
   <xacro:arg name="dynamixel_config_file" default="NOT_SET_2" />
-  -->
   <link name="world">
   </link>
@@ -128,4 +126,8 @@
    <child link="l_hand_link"/>
   </joint>
-  <xacro:robot name="Robot"/>
+  <xacro:robot name="Robot" prefix=""
+    use_fake_hardware="$(arg use_fake_hardware)"
+    fake_sensor_commands="$(arg fake_sensor_commands)"
+    slowdown="$(arg slowdown)"
+    dynamixel_config_file="$(arg dynamixel_config_file)"/>
 </robot>

File: src/inmoov_description/robots/robot.ros2_control.xacro (robot description, xacro)
@@ -1,11 +1,19 @@
 <?xml version="1.0"?>
 <robot xmlns:xacro="http://www.ros.org/wiki/xacro">
-  <xacro:macro name="robot" params="name">
+  <xacro:macro name="robot" params="name prefix use_fake_hardware:=^|true fake_sensor_commands:=^|false slowdown:=2.0 dynamixel_config_file">
     <ros2_control name="${name}" type="system">
       <hardware>
-        <plugin>dynamixel_hardware/DynamixelHardware</plugin>
+        <xacro:if value="${use_fake_hardware}">
+          <plugin>fake_components/GenericSystem</plugin>
+          <param name="fake_sensor_commands">${fake_sensor_commands}</param>
+          <param name="state_following_offset">0.0</param>
+        </xacro:if>
+        <xacro:unless value="${use_fake_hardware}">
+        <plugin>robot_hardware/RobotHardware</plugin>
+        <param name="dynamixel_info">${dynamixel_config_file}</param>
         <param name="usb_port">/dev/ttyUSB0</param>
         <param name="baud_rate">1000000</param>
-        <param name="use_dummy">true</param>
+        <param name="use_fake">true</param>
+        </xacro:unless>
       </hardware>
       <joint name="head_jaw_joint">

Commit message: fake robot launch made to work right and cleaned things up

File: src/inmoov_description/robots/inmoov.urdf.xacro (robot description, xacro)
@@ -18,8 +18,6 @@
     <origin xyz="0 0 0" rpy="0 0 0" />
   </xacro:rrbot>-->
-  <xacro:arg name="fake_sensor_commands" default="true" />
   <xacro:arg name="use_fake_hardware" default="true" />
   <xacro:arg name="prefix" default="" />
-  <xacro:arg name="slowdown" default="2.0" />
   <xacro:arg name="dynamixel_config_file" default="NOT_SET_2" />
   <link name="world">
@@ -128,6 +126,4 @@
   <xacro:robot name="Robot" prefix=""
     use_fake_hardware="$(arg use_fake_hardware)"
-    fake_sensor_commands="$(arg fake_sensor_commands)"
-    slowdown="$(arg slowdown)"
     dynamixel_config_file="$(arg dynamixel_config_file)"/>
 </robot>

File: src/inmoov_description/robots/robot.ros2_control.xacro (robot description, xacro)
@@ -1,18 +1,15 @@
 <?xml version="1.0"?>
 <robot xmlns:xacro="http://www.ros.org/wiki/xacro">
-  <xacro:macro name="robot" params="name prefix use_fake_hardware:=^|true fake_sensor_commands:=^|false slowdown:=2.0 dynamixel_config_file">
+  <xacro:macro name="robot" params="name prefix use_fake_hardware:=^|true dynamixel_config_file">
     <ros2_control name="${name}" type="system">
       <hardware>
+        <plugin>robot_hardware/RobotHardware</plugin>
         <xacro:if value="${use_fake_hardware}">
-          <plugin>fake_components/GenericSystem</plugin>
-          <param name="fake_sensor_commands">${fake_sensor_commands}</param>
-          <param name="state_following_offset">0.0</param>
+          <param name="use_fake">true</param>
         </xacro:if>
         <xacro:unless value="${use_fake_hardware}">
-        <plugin>robot_hardware/RobotHardware</plugin>
-        <param name="dynamixel_info">${dynamixel_config_file}</param>
-        <param name="usb_port">/dev/ttyUSB0</param>
-        <param name="baud_rate">57600</param>
-        <!--<param name="use_fake">true</param>-->
+          <param name="dynamixel_info">${dynamixel_config_file}</param>
+          <param name="usb_port">/dev/ttyUSB0</param>
+          <param name="baud_rate">57600</param>
         </xacro:unless>
       </hardware>
