Commit message: Shoulder's added to simulator with angles converted from degrees to rad

File: src/inmoov_description/robots/inmoov.urdf.xacro (robot description, xacro)
@@ -92,8 +92,17 @@
     <child link="face_link"/>
   </joint>
+  <xacro:property name="r_wrist_roll_joint_neutral_yaw" value="0.0" />
+  <xacro:property name="l_wrist_roll_joint_neutral_yaw" value="0.0" />
+  <xacro:property name="r_shoulder_out_joint_type" value="revolute" />
+  <xacro:property name="l_shoulder_out_joint_type" value="revolute" />
+  <xacro:if value="$(arg use_fake_hardware)">
+    <xacro:include filename="$(find inmoov_description)/urdf/shoulder_simulation.urdf.xacro" />
+  </xacro:if>
   <xacro:arm side="r" flip="1" covers="yes" />
-  <joint name="r_shoulder_out_joint" type="revolute">
-   <axis xyz="1 0 0"/>
-   <limit effort="1000.0" lower="${r_shoulder_out_joint_lower}" upper="${r_shoulder_out_joint_upper}" velocity="${r_shoulder_out_joint_velocity}" />
+  <joint name="r_shoulder_out_joint" type="${r_shoulder_out_joint_type}">
+   <xacro:if value="${r_shoulder_out_joint_type == 'revolute'}">
+    <axis xyz="1 0 0"/>
+    <limit effort="1000.0" lower="${r_shoulder_out_joint_lower}" upper="${r_shoulder_out_joint_upper}" velocity="${r_shoulder_out_joint_velocity}" />
+   </xacro:if>
    <origin rpy="0 0 0" xyz="0 -0.143 0.298"/>
    <parent link="torso_link"/>
@@ -104,12 +113,14 @@
    <axis xyz="0 0 1"/>
    <limit effort="1000.0" lower="${r_wrist_roll_joint_lower}" upper="${r_wrist_roll_joint_upper}" velocity="${r_wrist_roll_joint_velocity}" />
-   <origin rpy="0 0 0" xyz="-0.0144 0.01  -0.2885"/>
+   <origin rpy="0 0 ${r_wrist_roll_joint_neutral_yaw}" xyz="-0.0144 0.01  -0.2885"/>
    <parent link="r_forearm_link"/>
    <child link="r_hand_link"/>
   </joint>
   <xacro:arm side="l" flip="-1" covers="yes" />
-  <joint name="l_shoulder_out_joint" type="revolute">
-   <axis xyz="1 0 0"/>
-   <limit effort="1000.0" lower="${l_shoulder_out_joint_lower}" upper="${l_shoulder_out_joint_upper}" velocity="${l_shoulder_out_joint_velocity}" />
+  <joint name="l_shoulder_out_joint" type="${l_shoulder_out_joint_type}">
+   <xacro:if value="${l_shoulder_out_joint_type == 'revolute'}">
+    <axis xyz="1 0 0"/>
+    <limit effort="1000.0" lower="${l_shoulder_out_joint_lower}" upper="${l_shoulder_out_joint_upper}" velocity="${l_shoulder_out_joint_velocity}" />
+   </xacro:if>
    <origin rpy="0 0 0" xyz="0 0.143 0.298"/>
    <parent link="torso_link"/>
@@ -120,5 +131,5 @@
    <axis xyz="0 0 1"/>
    <limit effort="1000.0" lower="${l_wrist_roll_joint_lower}" upper="${l_wrist_roll_joint_upper}" velocity="${l_wrist_roll_joint_velocity}" />
-   <origin rpy="0 0 0" xyz="-0.0144 -0.01  -0.2885"/>
+   <origin rpy="0 0 ${l_wrist_roll_joint_neutral_yaw}" xyz="-0.0144 -0.01  -0.2885"/>
    <parent link="l_forearm_link"/>
    <child link="l_hand_link"/>

File: src/inmoov_description/robots/robot.ros2_control.xacro (robot description, xacro)
@@ -1,4 +1,11 @@
 <?xml version="1.0"?>
 <robot xmlns:xacro="http://www.ros.org/wiki/xacro">
+  <xacro:macro name="simulated_arm_interface" params="joint">
+    <joint name="${joint}">
+      <command_interface name="position"/>
+      <state_interface name="position"/>
+      <state_interface name="velocity"/>
+    </joint>
+  </xacro:macro>
   <xacro:macro name="robot" params="name prefix use_fake_hardware:=^|true dynamixel_config_file">
     <ros2_control name="${name}" type="system">
@@ -57,9 +64,20 @@
         <state_interface name="velocity"/>
       </joint>
-      <joint name="r_shoulder_out_joint">
-        <command_interface name="position"/>
-        <state_interface name="position"/>
-        <state_interface name="velocity"/>
-      </joint>
+      <xacro:unless value="${use_fake_hardware}">
+        <joint name="r_shoulder_out_joint">
+          <command_interface name="position"/>
+          <state_interface name="position"/>
+          <state_interface name="velocity"/>
+        </joint>
+      </xacro:unless>
+      <xacro:if value="${use_fake_hardware}">
+        <xacro:simulated_arm_interface joint="r_upper_arm_roll_joint"/>
+        <xacro:simulated_arm_interface joint="r_elbow_flex_joint"/>
+        <xacro:simulated_arm_interface joint="r_wrist_roll_joint"/>
+        <xacro:simulated_arm_interface joint="l_shoulder_lift_joint"/>
+        <xacro:simulated_arm_interface joint="l_upper_arm_roll_joint"/>
+        <xacro:simulated_arm_interface joint="l_elbow_flex_joint"/>
+        <xacro:simulated_arm_interface joint="l_wrist_roll_joint"/>
+      </xacro:if>
       <joint name="r_thumb_joint">
         <command_interface name="position"/>
