Commit message: Left hand to virtual robot, hand_gestures_node

File: src/inmoov_description/robots/robot.ros2_control.xacro (robot description, xacro)
@@ -126,4 +126,44 @@
         <state_interface name="velocity"/>
       </joint>
+      <joint name="l_thumb_joint">
+        <command_interface name="position">
+          <param name="min">-1</param>
+          <param name="max">1</param>
+        </command_interface>
+        <state_interface name="position"/>
+        <state_interface name="velocity"/>
+      </joint>
+      <joint name="l_index1_joint">
+        <command_interface name="position">
+          <param name="min">-1</param>
+          <param name="max">1</param>
+        </command_interface>
+        <state_interface name="position"/>
+        <state_interface name="velocity"/>
+      </joint>
+      <joint name="l_middle1_joint">
+        <command_interface name="position">
+          <param name="min">-1</param>
+          <param name="max">1</param>
+        </command_interface>
+        <state_interface name="position"/>
+        <state_interface name="velocity"/>
+      </joint>
+      <joint name="l_ring_joint">
+        <command_interface name="position">
+          <param name="min">-1</param>
+          <param name="max">1</param>
+        </command_interface>
+        <state_interface name="position"/>
+        <state_interface name="velocity"/>
+      </joint>
+      <joint name="l_pinky_joint">
+        <command_interface name="position">
+          <param name="min">-1</param>
+          <param name="max">1</param>
+        </command_interface>
+        <state_interface name="position"/>
+        <state_interface name="velocity"/>
+      </joint>
     </ros2_control>
   </xacro:macro>

Commit message: depency updates or fixes

File: src/inmoov_description/robots/robot.ros2_control.xacro (robot description, xacro)
@@ -9,4 +9,5 @@
         </xacro:if>
         <xacro:unless value="${use_fake_hardware}">
+          <param name="use_fake">false</param>
           <param name="dynamixel_info">${dynamixel_config_file}</param>
           <param name="usb_port">/dev/ttyUSB0</param>
@@ -14,9 +15,9 @@
         </xacro:unless>
       </hardware>
-      <joint name="head_jaw_joint">
+      <!--joint name="head_jaw_joint">
         <command_interface name="position"/>
         <state_interface name="position"/>
         <state_interface name="velocity"/>
-      </joint>
+      </joint-->
       <joint name="head_pan_joint">
         <command_interface name="position"/>

Commit message: added options for future dev

File: src/inmoov_description/robots/robot.ros2_control.xacro (robot description, xacro)
@@ -15,9 +15,9 @@
         </xacro:unless>
       </hardware>
-      <!--joint name="head_jaw_joint">
+      <joint name="head_jaw_joint">
         <command_interface name="position"/>
         <state_interface name="position"/>
         <state_interface name="velocity"/>
-      </joint-->
+      </joint>
       <joint name="head_pan_joint">
         <command_interface name="position"/>
@@ -56,4 +56,34 @@
       </joint>
       <joint name="r_shoulder_out_joint">
+        <command_interface name="position"/>
+        <state_interface name="position"/>
+        <state_interface name="velocity"/>
+      </joint>
+      <joint name="r_upper_arm_roll_joint">
+        <command_interface name="position"/>
+        <state_interface name="position"/>
+        <state_interface name="velocity"/>
+      </joint>
+      <joint name="r_elbow_flex_joint">
+        <command_interface name="position"/>
+        <state_interface name="position"/>
+        <state_interface name="velocity"/>
+      </joint>
+      <joint name="l_shoulder_lift_joint">
+        <command_interface name="position"/>
+        <state_interface name="position"/>
+        <state_interface name="velocity"/>
+      </joint>
+      <joint name="l_shoulder_out_joint">
+        <command_interface name="position"/>
+        <state_interface name="position"/>
+        <state_interface name="velocity"/>
+      </joint>
+      <joint name="l_upper_arm_roll_joint">
+        <command_interface name="position"/>
+        <state_interface name="position"/>
+        <state_interface name="velocity"/>
+      </joint>
+      <joint name="l_elbow_flex_joint">
         <command_interface name="position"/>
         <state_interface name="position"/>

Commit message: testing using pixi as package manager and updated to ros2 jazzy

File: src/inmoov_description/robots/robot.ros2_control.xacro (robot description, xacro)
@@ -15,9 +15,9 @@
         </xacro:unless>
       </hardware>
-      <!--joint name="head_jaw_joint">
+      <joint name="head_jaw_joint">
         <command_interface name="position"/>
         <state_interface name="position"/>
         <state_interface name="velocity"/>
-      </joint-->
+      </joint>
       <joint name="head_pan_joint">
         <command_interface name="position"/>
@@ -25,19 +25,19 @@
         <state_interface name="velocity"/>
       </joint>
-      <joint name="head_tilt_right_joint">
+      <!--<joint name="head_tilt_right_joint">
         <command_interface name="position"/>
         <state_interface name="position"/>
         <state_interface name="velocity"/>
-      </joint>
-      <joint name="head_tilt_left_joint">
+      </joint>-->
+      <!--<joint name="head_tilt_left_joint">
         <command_interface name="position"/>
         <state_interface name="position"/>
         <state_interface name="velocity"/>
-      </joint>
-      <joint name="head_tilt_vertical_joint">
+      </joint>-->
+      <!--<joint name="head_tilt_vertical_joint">
         <command_interface name="position"/>
         <state_interface name="position"/>
         <state_interface name="velocity"/>
-      </joint>
+      </joint>-->
       <joint name="eyes_shift_horizontal_joint">
         <command_interface name="position"/>
@@ -65,10 +65,10 @@
         <state_interface name="velocity"/>
       </joint>
-      <joint name="r_index1_joint">
+      <joint name="r_index_joint">
         <command_interface name="position"/>
         <state_interface name="position"/>
         <state_interface name="velocity"/>
       </joint>
-      <joint name="r_middle1_joint">
+      <joint name="r_middle_joint">
         <command_interface name="position"/>
         <state_interface name="position"/>
@@ -90,10 +90,10 @@
         <state_interface name="velocity"/>
       </joint>
-      <joint name="l_index1_joint">
+      <joint name="l_index_joint">
         <command_interface name="position"/>
         <state_interface name="position"/>
         <state_interface name="velocity"/>
       </joint>
-      <joint name="l_middle1_joint">
+      <joint name="l_middle_joint">
         <command_interface name="position"/>
         <state_interface name="position"/>

File: src/inmoov_description/urdf/asmHand.urdf.xacro (robot description, xacro)
@@ -212,5 +212,5 @@
         </xacro:if>
       <origin rpy="${flip * 0.1} 0 0" xyz="0 ${flip * 0.029} -0.0577"/>
-      <mimic joint="${side}_thumb_joint" multiplier="${flip *0.75}" offset="0"/>
+      <!--<mimic joint="${side}_thumb_joint" multiplier="${flip *0.75}" offset="0"/>-->
       <parent link="${side}_hand_link"/>
       <child link="${side}_thumb1_link"/>
@@ -237,5 +237,5 @@
         </xacro:if>
       <origin rpy="0 0 0" xyz="0 0 -0.035"/>
-      <mimic joint="${side}_thumb_joint" multiplier="1" offset="0"/>
+      <!--<mimic joint="${side}_thumb_joint" multiplier="1" offset="0"/>-->
       <parent link="${side}_thumb2_link"/>
       <child link="${side}_thumb3_link"/>
@@ -250,5 +250,5 @@
         </xacro:if>
       <origin rpy="${flip * 0.1} 0 0" xyz="-0.0015 ${flip * 0.0342}  -0.119"/>
-      <mimic joint="${side}_index_joint" multiplier="1" offset="0"/>
+      <!--<mimic joint="${side}_index_joint" multiplier="1" offset="0"/>-->
       <parent link="${side}_hand_link"/>
       <child link="${side}_index1_link"/>
@@ -275,5 +275,5 @@
         </xacro:if>
       <origin rpy="0 0 0" xyz="0 0 -0.024"/>
-      <mimic joint="${side}_index_joint" multiplier="1" offset="0"/>
+      <!--<mimic joint="${side}_index_joint" multiplier="1" offset="0"/>-->
       <parent link="${side}_index2_link"/>
       <child link="${side}_index3_link"/>
@@ -288,5 +288,5 @@
         </xacro:if>
       <origin rpy="0 0 0" xyz="-0.00175 ${flip * 0.007}  -0.12325"/>
-      <mimic joint="${side}_middle_joint" multiplier="1" offset="0"/>
+      <!--<mimic joint="${side}_middle_joint" multiplier="1" offset="0"/>-->
       <parent link="${side}_hand_link"/>
       <child link="${side}_middle1_link"/>
@@ -313,5 +313,5 @@
         </xacro:if>
       <origin rpy="0 0 0" xyz="0 0.0005 -0.0259"/>
-      <mimic joint="${side}_middle_joint" multiplier="1" offset="0"/>
+      <!--<mimic joint="${side}_middle_joint" multiplier="1" offset="0"/>-->
       <parent link="${side}_middle2_link"/>
       <child link="${side}_middle3_link"/>
@@ -326,5 +326,5 @@
         </xacro:if>
       <origin rpy="${flip * 0.7} 0 0" xyz="0 ${flip * -0.00705} -0.0794"/>
-      <mimic joint="${side}_ring_joint" multiplier="${flip * -0.1}" offset="0"/>
+      <!--<mimic joint="${side}_ring_joint" multiplier="${flip * -0.1}" offset="0"/>-->
       <parent link="${side}_hand_link"/>
       <child link="${side}_ring1_link"/>
@@ -351,5 +351,5 @@
         </xacro:if>
       <origin rpy="0 0 0" xyz="0 0.0005 -0.0345"/>
-      <mimic joint="${side}_ring_joint" multiplier="1" offset="0"/>
+      <!--<mimic joint="${side}_ring_joint" multiplier="1" offset="0"/>-->
       <parent link="${side}_ring2_link"/>
       <child link="${side}_ring3_link"/>
@@ -364,5 +364,5 @@
         </xacro:if>
       <origin rpy="0 0 0" xyz="0 0.0004 -0.0229"/>
-      <mimic joint="${side}_ring_joint" multiplier="1" offset="0"/>
+      <!--<mimic joint="${side}_ring_joint" multiplier="1" offset="0"/>-->
       <parent link="${side}_ring3_link"/>
       <child link="${side}_ring4_link"/>
@@ -377,5 +377,5 @@
         </xacro:if>
       <origin rpy="${flip * 0.7} 0 0" xyz="0 ${flip * -0.0270} -0.0555"/>
-      <mimic joint="${side}_pinky_joint" multiplier="${flip * -0.1}" offset="0"/>
+      <!--<mimic joint="${side}_pinky_joint" multiplier="${flip * -0.1}" offset="0"/>-->
       <parent link="${side}_hand_link"/>
       <child link="${side}_pinky1_link"/>
@@ -402,5 +402,5 @@
         </xacro:if>
       <origin rpy="0 0 0" xyz="0 0.0005 -0.031"/>
-      <mimic joint="${side}_pinky_joint" multiplier="1" offset="0"/>
+      <!--<mimic joint="${side}_pinky_joint" multiplier="1" offset="0"/>-->
       <parent link="${side}_pinky2_link"/>
       <child link="${side}_pinky3_link"/>
@@ -415,5 +415,5 @@
         </xacro:if>
       <origin rpy="0 0 0" xyz="0 0.0004 -0.0208"/>
-      <mimic joint="${side}_pinky_joint" multiplier="1" offset="0"/>
+      <!--<mimic joint="${side}_pinky_joint" multiplier="1" offset="0"/>-->
       <parent link="${side}_pinky3_link"/>
       <child link="${side}_pinky4_link"/>

File: src/inmoov_description/urdf/inmoov-moveit-gazebo.urdf (robot description, URDF)
Before this commit: robot inmoov, 90 links, 89 joints
Joints:
- joint l_index1_joint: mimic joint=l_index_joint multiplier=1 offset=0 -> (none)
- joint l_index3_joint: mimic joint=l_index_joint multiplier=1 offset=0 -> (none)
- joint l_middle1_joint: mimic joint=l_middle_joint multiplier=1 offset=0 -> (none)
- joint l_middle3_joint: mimic joint=l_middle_joint multiplier=1 offset=0 -> (none)
- joint l_pinky1_joint: mimic joint=l_pinky_joint multiplier=0.1 offset=0 -> (none)
- joint l_pinky3_joint: mimic joint=l_pinky_joint multiplier=1 offset=0 -> (none)
- joint l_pinky4_joint: mimic joint=l_pinky_joint multiplier=1 offset=0 -> (none)
- joint l_ring1_joint: mimic joint=l_ring_joint multiplier=0.1 offset=0 -> (none)
- joint l_ring3_joint: mimic joint=l_ring_joint multiplier=1 offset=0 -> (none)
- joint l_ring4_joint: mimic joint=l_ring_joint multiplier=1 offset=0 -> (none)
- joint l_thumb1_joint: mimic joint=l_thumb_joint multiplier=-0.75 offset=0 -> (none)
- joint l_thumb3_joint: mimic joint=l_thumb_joint multiplier=1 offset=0 -> (none)
- joint r_index1_joint: mimic joint=r_index_joint multiplier=1 offset=0 -> (none)
- joint r_index3_joint: mimic joint=r_index_joint multiplier=1 offset=0 -> (none)
- joint r_middle1_joint: mimic joint=r_middle_joint multiplier=1 offset=0 -> (none)
- joint r_middle3_joint: mimic joint=r_middle_joint multiplier=1 offset=0 -> (none)
- joint r_pinky1_joint: mimic joint=r_pinky_joint multiplier=-0.1 offset=0 -> (none)
- joint r_pinky3_joint: mimic joint=r_pinky_joint multiplier=1 offset=0 -> (none)
- joint r_pinky4_joint: mimic joint=r_pinky_joint multiplier=1 offset=0 -> (none)
- joint r_ring1_joint: mimic joint=r_ring_joint multiplier=-0.1 offset=0 -> (none)
- joint r_ring3_joint: mimic joint=r_ring_joint multiplier=1 offset=0 -> (none)
- joint r_ring4_joint: mimic joint=r_ring_joint multiplier=1 offset=0 -> (none)
- joint r_thumb3_joint: mimic joint=r_thumb_joint multiplier=1 offset=0 -> (none)

Commit message: fixes

File: src/inmoov_description/robots/robot.ros2_control.xacro (robot description, xacro)
@@ -15,9 +15,9 @@
         </xacro:unless>
       </hardware>
-      <!--joint name="head_jaw_joint">
+      <joint name="head_jaw_joint">
         <command_interface name="position"/>
         <state_interface name="position"/>
         <state_interface name="velocity"/>
-      </joint-->
+      </joint>
       <joint name="head_pan_joint">
         <command_interface name="position"/>
