Commit message: changed launch demo to a ros2 launch file, unified_arms node now in separate package, jaw controller fixes, speach_recognizer node replaced with stt node for better performance, qabot replaced with llm node which uses openai generic client

File: src/inmoov_description/robots/robot.ros2_control.xacro (robot description, xacro)
@@ -15,9 +15,11 @@
         </xacro:unless>
       </hardware>
-      <!--joint name="head_jaw_joint">
-        <command_interface name="position"/>
-        <state_interface name="position"/>
-        <state_interface name="velocity"/>
-      </joint-->
+      <xacro:if value="${use_fake_hardware}">
+        <joint name="head_jaw_joint">
+          <command_interface name="position"/>
+          <state_interface name="position"/>
+          <state_interface name="velocity"/>
+        </joint>
+      </xacro:if>
       <joint name="head_pan_joint">
         <command_interface name="position"/>
