Commit message: Remove redundant files, add "follow joint trajectory action" server and "turn_head" test script.
Note: currently tries to execute joints that have no servos, so servo controller crashes

File: src/inmoov_description/urdf/config.joints.urdf.xacro (robot description, xacro)
@@ -1,5 +1,5 @@
 <?xml version="1.0"?>
 <robot xmlns:xacro="http://ros.org/wiki/xacro">
-  <xacro:property name="filename" value="$(find inmoov_bringup)/config/config.yaml"/>
+  <xacro:property name="filename" value="$(find inmoov_description)/config/config.yaml"/>
   <xacro:property name="c" value="${load_yaml(filename)}"/>
   <!--xacro:property name="pi" value="3.1415926539"/-->

Commit message: WIP update launchsettings
* rename spawner.py to only spawner
* prefix with xacro to load_yaml files

File: src/inmoov_description/urdf/config.joints.urdf.xacro (robot description, xacro)
@@ -2,5 +2,5 @@
 <robot xmlns:xacro="http://ros.org/wiki/xacro">
   <xacro:property name="filename" value="$(find inmoov_description)/config/config.yaml"/>
-  <xacro:property name="c" value="${load_yaml(filename)}"/>
+  <xacro:property name="c" value="${xacro.load_yaml(filename)}"/>
   <!--xacro:property name="pi" value="3.1415926539"/-->
   <xacro:if value="${c['bringup']['angles'] == 'degrees'}">
