Commit message: fixed left hand simulation position

File: src/inmoov_description/urdf/asmHand.urdf.xacro (robot description, xacro)
@@ -250,5 +250,4 @@
         </xacro:if>
       <origin rpy="${flip * 0.1} 0 0" xyz="-0.0015 ${flip * 0.0342}  -0.119"/>
-      <mimic joint="${side}_index_joint" multiplier="1" offset="0"/>
       <parent link="${side}_hand_link"/>
       <child link="${side}_index1_link"/>
@@ -263,4 +262,5 @@
         </xacro:if>
       <origin rpy="0 0 0" xyz="0 0.001 -0.03595"/>
+      <mimic joint="${side}_index1_joint" multiplier="1" offset="0"/>
       <parent link="${side}_index1_link"/>
       <child link="${side}_index2_link"/>
@@ -275,5 +275,5 @@
         </xacro:if>
       <origin rpy="0 0 0" xyz="0 0 -0.024"/>
-      <mimic joint="${side}_index_joint" multiplier="1" offset="0"/>
+      <mimic joint="${side}_index1_joint" multiplier="1" offset="0"/>
       <parent link="${side}_index2_link"/>
       <child link="${side}_index3_link"/>
@@ -288,5 +288,4 @@
         </xacro:if>
       <origin rpy="0 0 0" xyz="-0.00175 ${flip * 0.007}  -0.12325"/>
-      <mimic joint="${side}_middle_joint" multiplier="1" offset="0"/>
       <parent link="${side}_hand_link"/>
       <child link="${side}_middle1_link"/>
@@ -301,4 +300,5 @@
         </xacro:if>
       <origin rpy="0 0 0" xyz="0 0.000 -0.0389"/>
+      <mimic joint="${side}_middle1_joint" multiplier="1" offset="0"/>
       <parent link="${side}_middle1_link"/>
       <child link="${side}_middle2_link"/>
@@ -313,5 +313,5 @@
         </xacro:if>
       <origin rpy="0 0 0" xyz="0 0.0005 -0.0259"/>
-      <mimic joint="${side}_middle_joint" multiplier="1" offset="0"/>
+      <mimic joint="${side}_middle1_joint" multiplier="1" offset="0"/>
       <parent link="${side}_middle2_link"/>
       <child link="${side}_middle3_link"/>
