Commit message: refactor(robot): group motion and description packages
Move hardware, motion, and InMoov description packages into subsystem directories. Add sop_robot_common for shared robot contracts, calibration, and arm action helpers, and keep console entrypoints on package-root node modules for motion bridges.

File: src/sop_robot_description/inmoov_description/robots/robot.ros2_control.xacro (robot description, xacro)
@@ -55,5 +55,35 @@
         <state_interface name="velocity"/>
       </joint>
+      <joint name="r_upper_arm_roll_joint">
+        <command_interface name="position"/>
+        <state_interface name="position"/>
+        <state_interface name="velocity"/>
+      </joint>
+      <joint name="r_elbow_flex_joint">
+        <command_interface name="position"/>
+        <state_interface name="position"/>
+        <state_interface name="velocity"/>
+      </joint>
       <joint name="r_shoulder_out_joint">
+        <command_interface name="position"/>
+        <state_interface name="position"/>
+        <state_interface name="velocity"/>
+      </joint>
+      <joint name="l_shoulder_lift_joint">
+        <command_interface name="position"/>
+        <state_interface name="position"/>
+        <state_interface name="velocity"/>
+      </joint>
+      <joint name="l_upper_arm_roll_joint">
+        <command_interface name="position"/>
+        <state_interface name="position"/>
+        <state_interface name="velocity"/>
+      </joint>
+      <joint name="l_elbow_flex_joint">
+        <command_interface name="position"/>
+        <state_interface name="position"/>
+        <state_interface name="velocity"/>
+      </joint>
+      <joint name="l_shoulder_out_joint">
         <command_interface name="position"/>
         <state_interface name="position"/>
